File: hardware/weather station.kicad_pcb (KiCad board)
At the start: 2 copper layers, 95 x 72 mm, 54 parts, among them J1 Solar Panel, J10 Pressure, J11 Conn_01x04, J12 Conn_02x07_Odd_Even, J2 DIG_EXP, J3 ICSP, J4 BAT., J5 EXP0, J6 EXP1, J7 Wind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

Commit message: pcb layout complete
Parts:
- added REF**: OSHW-Logo2_7.3x6mm_SilkScreen, Symbol:OSHW-Logo2_7.3x6mm_SilkScreen, F.Cu at (120.9, 131.3)
- added REF**: MountingHole_3.2mm_M3, MountingHole:MountingHole_3.2mm_M3, F.Cu at (58.0, 131.0)
- added REF**: MountingHole_3.2mm_M3, MountingHole:MountingHole_3.2mm_M3, F.Cu at (58.0, 69.0)
- added REF**: MountingHole_3.2mm_M3, MountingHole:MountingHole_3.2mm_M3, F.Cu at (143.0, 69.0)
- added REF**: MountingHole_3.2mm_M3, MountingHole:MountingHole_3.2mm_M3, F.Cu at (143.0, 131.0)
- added REF**: WEEE-Logo_4.2x6mm_SilkScreen, Symbol:WEEE-Logo_4.2x6mm_SilkScreen, B.Cu at (67.7, 69.0)
- moved C11 309.1 mm to (92.2, 86.7), turned to 180 degrees
- moved R6 308.7 mm to (89.4, 96.7), turned to 90 degrees
- moved R10 308.0 mm to (93.8, 96.7), turned to 270 degrees
- moved R7 305.0 mm to (91.6, 96.7), turned to 270 degrees
- moved J7 300.0 mm to (58.6, 74.7)
- moved R17 285.2 mm to (110.7, 71.3)
- moved R5 284.9 mm to (98.3, 73.5), turned to 180 degrees
- moved R8 282.4 mm to (116.6, 100.8), turned to 90 degrees
- moved C10 280.3 mm to (105.3, 92.3), turned to 90 degrees
- moved C4 278.1 mm to (105.4, 109.6), turned to 270 degrees
- moved D5 273.9 mm to (111.9, 124.6), turned to 180 degrees
- moved R16 259.2 mm to (138.2, 76.7), turned to 180 degrees
- moved U5 258.5 mm to (92.2, 91.3)
- moved R11 258.4 mm to (117.3, 71.5)
- moved U4 256.2 mm to (112.1, 108.3)
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Routing:
- net +5V: track 0.00 -> 378.1 mm, vias 0 -> 11
- net PGD: track 0.00 -> 137.9 mm
- net PGC: track 0.00 -> 125.5 mm, vias 0 -> 1
- net VGND: track 0.00 -> 107.9 mm
- net SOLAR_PANEL: track 0.00 -> 88.4 mm, vias 0 -> 2
- net WIFI_BOOT: track 0.00 -> 79.0 mm, vias 0 -> 4
- net WIFI_READY: track 0.00 -> 73.7 mm, vias 0 -> 2
- net WIFI_RX: track 0.00 -> 73.2 mm, vias 0 -> 2
- net WIFI_RESET: track 0.00 -> 72.1 mm, vias 0 -> 2
- net WIFI_TX: track 0.00 -> 70.1 mm, vias 0 -> 2
- net CTRL1: track 0.00 -> 66.7 mm, vias 0 -> 2
- net Net-(J7-Pad4): track 0.00 -> 65.9 mm, vias 0 -> 2
- net CTRL0: track 0.00 -> 58.0 mm, vias 0 -> 2
- net Net-(J3-Pad1): track 0.00 -> 50.4 mm, vias 0 -> 1
- net Net-(C12-Pad1): track 0.00 -> 49.2 mm
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- added copper zone on B.Cu, net GND
- added copper zone on F.Cu, net GND
Other:
- net class +5V added: clearance 0.2, trace_width 0.4, via_dia 0.8, via_drill 0.4
- net class Power added: clearance 0.2, trace_width 1, via_dia 0.8, via_drill 0.4
- board text added: "Humidity"
- board text added: "ICSP"
- board text added: "Magnetic Field"
- board text added: "Pressure Temperature"
- board text added: "Taur 2018 http://taur-tech.com"
- board text added: "WIFI"
- board text added: "Weather Station rev. 2"
- board text added: "Wind"
- board text added: "http://taur-tech.com"
